Commit message: gripper

File: ur_description/urdf/ur5.xacro (robot description, xacro)
@@ -14,5 +14,55 @@
     Refer to 'inc/ur_macro.xacro' for more information.
   -->
-  <xacro:include filename="$(find ur_description)/urdf/inc/ur5_macro.xacro"/>
-  <xacro:ur5_robot prefix="" />
+  <xacro:macro name="ur5" params="ur5_prefix">
+    <xacro:include filename="$(find ur_description)/urdf/inc/ur5_macro.xacro"/>
+    <xacro:include filename="$(find ur_description)/urdf/eef.xacro"/>
+    <!-- Configure self collision properties per link -->
+    <gazebo reference="${ur5_prefix}shoulder_link">
+      <selfCollide>true</selfCollide>
+    </gazebo>
+    <gazebo reference="${ur5_prefix}upper_arm_link">
+      <selfCollide>true</selfCollide>
+    </gazebo>
+    <gazebo reference="${ur5_prefix}forearm_link">
+      <selfCollide>true</selfCollide>
+    </gazebo>
+    <gazebo reference="${ur5_prefix}wrist_1_link">
+      <selfCollide>true</selfCollide>
+    </gazebo>
+    <gazebo reference="${ur5_prefix}wrist_3_link">
+      <selfCollide>true</selfCollide>
+    </gazebo>
+    <gazebo reference="${ur5_prefix}wrist_2_link">
+      <selfCollide>true</selfCollide>
+    </gazebo>
+    <gazebo reference="${ur5_prefix}ee_link">
+      <selfCollide>true</selfCollide>
+    </gazebo>
+    <gazebo>
+     <plugin name="gazebo_grasp_fix" filename="libgazebo_grasp_fix.so">
+           <arm>
+             <arm_name>${ur5_prefix}ur5_gripper</arm_name>
+             <palm_link>${ur5_prefix}wrist_3_link</palm_link>
+             <gripper_link>${ur5_prefix}robotiq_85_base_link</gripper_link>
+             <gripper_link>${ur5_prefix}robotiq_85_left_knuckle_link</gripper_link>
+             <gripper_link>${ur5_prefix}robotiq_85_right_knuckle_link</gripper_link>
+             <gripper_link>${ur5_prefix}robotiq_85_left_finger_link</gripper_link>
+             <gripper_link>${ur5_prefix}robotiq_85_right_finger_link</gripper_link>
+             <gripper_link>${ur5_prefix}robotiq_85_left_inner_knuckle_link</gripper_link>
+             <gripper_link>${ur5_prefix}robotiq_85_right_inner_knuckle_link</gripper_link>
+             <gripper_link>${ur5_prefix}robotiq_85_left_finger_tip_link</gripper_link>
+             <gripper_link>${ur5_prefix}robotiq_85_right_finger_tip_link</gripper_link>
+           </arm>
+       <forces_angle_tolerance>150</forces_angle_tolerance>
+       <update_rate>130</update_rate>
+       <grip_count_threshold>2</grip_count_threshold>
+       <max_grip_count>8</max_grip_count>
+       <release_tolerance>0.01</release_tolerance>
+       <disable_collisions_on_attach>true</disable_collisions_on_attach>
+       <contact_topic>__default_topic__</contact_topic>
+     </plugin>
+   </gazebo>
+    <xacro:ur5_robot prefix="${ur5_prefix}" />
+    <xacro:robotiq_85_gripper ur5_prefix="${ur5_prefix}"/>
+  </xacro:macro>
 </robot>

Commit message: add d435

File: ur_description/urdf/ur5.xacro (robot description, xacro)
@@ -17,4 +17,8 @@
     <xacro:include filename="$(find ur_description)/urdf/inc/ur5_macro.xacro"/>
     <xacro:include filename="$(find ur_description)/urdf/eef.xacro"/>
+    <xacro:include filename="$(find realsense_ros_gazebo)/xacro/depthcam.xacro"/>
+    <xacro:realsense_d435 sensor_name="${ur5_prefix}" parent_link="${ur5_prefix}wrist_3_link" rate="30">
+      <origin rpy="1.57 -1.57 0" xyz="0 -0.1 0.0"/>
+    </xacro:realsense_d435>
     <!-- Configure self collision properties per link -->
     <gazebo reference="${ur5_prefix}shoulder_link">
